File: ICED - Right/ICEDRight.kicad_pcb (KiCad board)
At the start: 2 copper layers, 175.4 x 145 mm, 164 parts, among them P1 FLASH_HDR, P2 USBC, P3 CONN_17, P4 USB3_AFEMALE, Q1 TC1264, U1 MK20DX256VLH7, U2 IS31FL3731C, X1 CRYSTAL

Commit message: version stamp
Other:
- board text added: "ICEH-R Rev 3.4a Batch __"
- board text removed: "ICED-R Rev 1.2b Batch __"
Changed lines of the file:
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@@
   (page A4)
   (title_block
-    (title ICED-R)
-    (date 2016-07-17)
-    (rev "Rev 1.2b")
-    (company "Input Club")
+    (title ICEH-R)
+    (date 2017-05-14)
+    (rev 3.4a)
+    (company "ErgoHack")
   )
   (layers
@@
   (gr_line (start 110.7694 46.9392) (end 110.7694 43.18) (angle 90) (layer Edge.Cuts) (width 0.127))
   (gr_line (start 101.8286 43.18) (end 101.8286 46.9392) (angle 90) (layer Edge.Cuts) (width 0.127))
-  (gr_text "ICED-R Rev 1.2b Batch __" (at 133.35 52.578) (layer B.SilkS)
+  (gr_text "ICEH-R Rev 3.4a Batch __" (at 133.35 52.578) (layer B.SilkS)
     (effects (font (size 2 1.5) (thickness 0.3)) (justify mirror))
   )
